Commit message: feat: add hardware driver and bringup packages for real robot control
- Add alicia_m_driver package with ros2_control hardware interface
- Add alicia_m_bringup package with launch files
- Update alicia_m_moveit_config for hardware support

File: alicia_m_moveit_config/config/alicia_m_v1_1_follower.ros2_control.xacro (robot description, xacro)
@@ -1,10 +1,21 @@
 <?xml version="1.0"?>
 <robot xmlns:xacro="http://www.ros.org/wiki/xacro">
-    <xacro:macro name="alicia_m_v1_1_follower_ros2_control" params="name initial_positions_file">
-        <xacro:property name="initial_positions" value="${load_yaml(initial_positions_file)['initial_positions']}"/>
+    <xacro:macro name="alicia_m_v1_1_follower_ros2_control"
+                 params="name initial_positions_file
+                         ros2_control_plugin:='mock_components/GenericSystem'
+                         serial_port:='/dev/ttyACM0'
+                         baudrate:='1000000'
+                         control_mode:='pv'
+                         default_speed:='1.0'">
+        <xacro:property name="initial_positions" value="${xacro.load_yaml(initial_positions_file)['initial_positions']}"/>
         <ros2_control name="${name}" type="system">
             <hardware>
-                <!-- By default, set up controllers for simulation. This won't work on real hardware -->
-                <plugin>mock_components/GenericSystem</plugin>
+                <plugin>${ros2_control_plugin}</plugin>
+                <xacro:unless value="${ros2_control_plugin == 'mock_components/GenericSystem'}">
+                    <param name="serial_port">${serial_port}</param>
+                    <param name="baudrate">${baudrate}</param>
+                    <param name="control_mode">${control_mode}</param>
+                    <param name="default_speed">${default_speed}</param>
+                </xacro:unless>
             </hardware>
             <joint name="joint1">

File: alicia_m_moveit_config/config/alicia_m_v1_1_follower.urdf.xacro (robot description, xacro)
@@ -2,8 +2,20 @@
 <robot xmlns:xacro="http://www.ros.org/wiki/xacro" name="alicia_m_v1_1_follower">
     <xacro:arg name="initial_positions_file" default="initial_positions.yaml" />
-    <!-- Import alicia_m_v1_1_follower urdf file -->
+    <xacro:arg name="ros2_control_plugin" default="mock_components/GenericSystem" />
+    <xacro:arg name="serial_port" default="/dev/ttyACM0" />
+    <xacro:arg name="baudrate" default="1000000" />
+    <xacro:arg name="control_mode" default="pv" />
+    <xacro:arg name="default_speed" default="1.0" />
+    <!-- 导入 URDF 模型 -->
     <xacro:include filename="$(find alicia_m_descriptions)/urdf/Alicia_M_v1_1/Alicia_M_v1_1_follower.urdf" />
-    <!-- Import control_xacro -->
+    <!-- 导入 ros2_control 配置 -->
     <xacro:include filename="alicia_m_v1_1_follower.ros2_control.xacro" />
-    <xacro:alicia_m_v1_1_follower_ros2_control name="FakeSystem" initial_positions_file="$(arg initial_positions_file)"/>
+    <xacro:alicia_m_v1_1_follower_ros2_control
+        name="AliciaHardware"
+        initial_positions_file="$(arg initial_positions_file)"
+        ros2_control_plugin="$(arg ros2_control_plugin)"
+        serial_port="$(arg serial_port)"
+        baudrate="$(arg baudrate)"
+        control_mode="$(arg control_mode)"
+        default_speed="$(arg default_speed)"/>
 </robot>
